Commit message: lenny_moveit_config added and deleted from Lenny_Motoman packages

File: lenny_description/urdf/robotiq_85_gripper.urdf.xacro (robot description, xacro)
@@ -1,5 +1,5 @@
 <?xml version="1.0"?>
 <robot name="robotiq_85_gripper" xmlns:xacro="http://ros.org/wiki/xacro">
-    <xacro:include filename="$(find robotiq_85_description)/urdf/robotiq_85_gripper.transmission.xacro" />
+    <xacro:include filename="$(find lenny_description)/urdf/robotiq_85_gripper.transmission.xacro" />
     <xacro:property name="pi" value="3.14159"/>
     <xacro:macro name="robotiq_85_gripper" params="prefix parent *origin">
@@ -12,10 +12,10 @@
             <visual>
                 <geometry>
-                    <mesh filename="package://robotiq_85_description/meshes/visual/robotiq_85_base_link.dae"/>
-                </geometry>
-            </visual>
-            <collision>
-                <geometry>
-                    <mesh filename="package://robotiq_85_description/meshes/collision/robotiq_85_base_link.stl"/>
+                    <mesh filename="package://lenny_description/meshes/robotiq/visual/robotiq_85_base_link.dae"/>
+                </geometry>
+            </visual>
+            <collision>
+                <geometry>
+                    <mesh filename="package://lenny_description/meshes/robotiq/collision/robotiq_85_base_link.stl"/>
                 </geometry>
             </collision>
@@ -46,10 +46,10 @@
             <visual>
                 <geometry>
-                    <mesh filename="package://robotiq_85_description/meshes/visual/robotiq_85_knuckle_link.dae"/>
-                </geometry>
-            </visual>
-            <collision>
-                <geometry>
-                    <mesh filename="package://robotiq_85_description/meshes/collision/robotiq_85_knuckle_link.stl"/>
+                    <mesh filename="package://lenny_description/meshes/robotiq/visual/robotiq_85_knuckle_link.dae"/>
+                </geometry>
+            </visual>
+            <collision>
+                <geometry>
+                    <mesh filename="package://lenny_description/meshes/robotiq/collision/robotiq_85_knuckle_link.stl"/>
                 </geometry>
             </collision>
@@ -65,10 +65,10 @@
             <visual>
                 <geometry>
-                    <mesh filename="package://robotiq_85_description/meshes/visual/robotiq_85_knuckle_link.dae"/>
-                </geometry>
-            </visual>
-            <collision>
-                <geometry>
-                    <mesh filename="package://robotiq_85_description/meshes/collision/robotiq_85_knuckle_link.stl"/>
+                    <mesh filename="package://lenny_description/meshes/robotiq/visual/robotiq_85_knuckle_link.dae"/>
+                </geometry>
+            </visual>
+            <collision>
+                <geometry>
+                    <mesh filename="package://lenny_description/meshes/robotiq/collision/robotiq_85_knuckle_link.stl"/>
                 </geometry>
             </collision>
@@ -94,10 +94,10 @@
             <visual>
                 <geometry>
-                    <mesh filename="package://robotiq_85_description/meshes/visual/robotiq_85_finger_link.dae"/>
-                </geometry>
-            </visual>
-            <collision>
-                <geometry>
-                    <mesh filename="package://robotiq_85_description/meshes/collision/robotiq_85_finger_link.stl"/>
+                    <mesh filename="package://lenny_description/meshes/robotiq/visual/robotiq_85_finger_link.dae"/>
+                </geometry>
+            </visual>
+            <collision>
+                <geometry>
+                    <mesh filename="package://lenny_description/meshes/robotiq/collision/robotiq_85_finger_link.stl"/>
                 </geometry>
             </collision>
@@ -113,10 +113,10 @@
             <visual>
                 <geometry>
-                    <mesh filename="package://robotiq_85_description/meshes/visual/robotiq_85_finger_link.dae"/>
-                </geometry>
-            </visual>
-            <collision>
-                <geometry>
-                    <mesh filename="package://robotiq_85_description/meshes/collision/robotiq_85_finger_link.stl"/>
+                    <mesh filename="package://lenny_description/meshes/robotiq/visual/robotiq_85_finger_link.dae"/>
+                </geometry>
+            </visual>
+            <collision>
+                <geometry>
+                    <mesh filename="package://lenny_description/meshes/robotiq/collision/robotiq_85_finger_link.stl"/>
                 </geometry>
             </collision>
@@ -148,10 +148,10 @@
             <visual>
                 <geometry>
-                    <mesh filename="package://robotiq_85_description/meshes/visual/robotiq_85_inner_knuckle_link.dae"/>
-                </geometry>
-            </visual>
-            <collision>
-                <geometry>
-                    <mesh filename="package://robotiq_85_description/meshes/collision/robotiq_85_inner_knuckle_link.stl"/>
+                    <mesh filename="package://lenny_description/meshes/robotiq/visual/robotiq_85_inner_knuckle_link.dae"/>
+                </geometry>
+            </visual>
+            <collision>
+                <geometry>
+                    <mesh filename="package://lenny_description/meshes/robotiq/collision/robotiq_85_inner_knuckle_link.stl"/>
                 </geometry>
             </collision>
@@ -167,10 +167,10 @@
             <visual>
                 <geometry>
-                    <mesh filename="package://robotiq_85_description/meshes/visual/robotiq_85_inner_knuckle_link.dae"/>
-                </geometry>
-            </visual>
-            <collision>
-                <geometry>
-                    <mesh filename="package://robotiq_85_description/meshes/collision/robotiq_85_inner_knuckle_link.stl"/>
+                    <mesh filename="package://lenny_description/meshes/robotiq/visual/robotiq_85_inner_knuckle_link.dae"/>
+                </geometry>
+            </visual>
+            <collision>
+                <geometry>
+                    <mesh filename="package://lenny_description/meshes/robotiq/collision/robotiq_85_inner_knuckle_link.stl"/>
                 </geometry>
             </collision>
@@ -202,10 +202,10 @@
             <visual>
                 <geometry>
-                    <mesh filename="package://robotiq_85_description/meshes/visual/robotiq_85_finger_tip_link.dae"/>
-                </geometry>
-            </visual>
-            <collision>
-                <geometry>
-                    <mesh filename="package://robotiq_85_description/meshes/collision/robotiq_85_finger_tip_link.stl"/>
+                    <mesh filename="package://lenny_description/meshes/robotiq/visual/robotiq_85_finger_tip_link.dae"/>
+                </geometry>
+            </visual>
+            <collision>
+                <geometry>
+                    <mesh filename="package://lenny_description/meshes/robotiq/collision/robotiq_85_finger_tip_link.stl"/>
                 </geometry>
             </collision>
@@ -221,10 +221,10 @@
             <visual>
                 <geometry>
-                    <mesh filename="package://robotiq_85_description/meshes/visual/robotiq_85_finger_tip_link.dae"/>
-                </geometry>
-            </visual>
-            <collision>
-                <geometry>
-                    <mesh filename="package://robotiq_85_description/meshes/collision/robotiq_85_finger_tip_link.stl"/>
+                    <mesh filename="package://lenny_description/meshes/robotiq/visual/robotiq_85_finger_tip_link.dae"/>
+                </geometry>
+            </visual>
+            <collision>
+                <geometry>
+                    <mesh filename="package://lenny_description/meshes/robotiq/collision/robotiq_85_finger_tip_link.stl"/>
                 </geometry>
             </collision>

File: lenny_description/urdf/robotiq_85_gripper.xacro (robot description, xacro)
@@ -1,5 +1,5 @@
 <?xml version="1.0" ?>
 <robot name="robotiq_85_gripper" xmlns:xacro="http://ros.org/wiki/xacro">
-    <xacro:include filename="$(find robotiq_85_description)/urdf/robotiq_85_gripper.urdf.xacro" />
+    <xacro:include filename="$(find lenny_description)/urdf/robotiq_85_gripper.urdf.xacro" />
     <gazebo>
         <plugin name="gazebo_ros_control" filename="libgazebo_ros_control.so">
